File: Theremin.kicad_sch (KiCad schematic)
At the start: 0 parts

Commit message: finished output and added sd card
Parts:
- added C17: C, symbol Device:C
- added J3: AudioJack3, symbol Connector_Audio:AudioJack3
- added R13: R_US, symbol Eclectronics:R_US
- added U3: MCP4725xxx-xCH, Package_TO_SOT_SMD:SOT-23-6, symbol Analog_DAC:MCP4725xxx-xCH
Connections:
- new net: C17.2, R13.1, U3.1 (VOUT)
- new net: C17.1, J3.R, J3.T
- new net: J3.S, R13.2
- new net +3V3: U3.3 (VDD)
- new net GND: U3.2 (VSS), U3.6 (A0)
- new net GPIO4: U3.4 (SDA)
- new net GPIO5: U3.5 (SCL)
